File: Docs/MICAS_Circuit/MICAS_Circuit.kicad_sch (KiCad schematic)
At the start: 34 parts, among them Q1 BD140, Q2 BD140, U1 ESP32_DevKit_V1_DOIT

Commit message: update repository with circuit data
Parts:
- removed MAX485_MOD1: ~, MAX485_Module:MAX485_MODULE, symbol MAX485_Module:MAX485
- removed MP2482_Module1: ~, MP2482_Module:MP2482_Module, symbol MP2482_Module:MP2482_Module
- removed NPK_SENSOR1: Screw_Terminal_01x04, TerminalBlock:TerminalBlock_bornier-4_P5.08mm, symbol Connector:Screw_Terminal_01x04
- removed POWER_SUPPLY1: Screw_Terminal_01x02, TerminalBlock:TerminalBlock_bornier-2_P5.08mm, symbol Connector:Screw_Terminal_01x02
- added 12V_PWR1: Screw_Terminal_01x02, KF301-2P:KF301-2P, symbol Connector:Screw_Terminal_01x02
- added D3: RLED, LED_THT:LED_D5.0mm_FlatTop, symbol Device:LED
- added D4: GLED, LED_THT:LED_D5.0mm_FlatTop, symbol Device:LED
- added D5: BLED, LED_THT:LED_D5.0mm_FlatTop, symbol Device:LED
- added MAX485MOD1: ~, MAX485_Module:MAX485_MOD, symbol MAX485_Module:MAX485_MOD
- added MP2482MOD1: ~, MP2482_Module:MP2482_MOD, symbol MP2482_Module:MP2482_MOD
- added NPK_SEN1: Screw_Terminal_01x04, TerminalBlock:TerminalBlock_Xinya_XY308-2.54-4P_1x04_P2.54mm_Horizontal, symbol Connector:Screw_Terminal_01x04
- added R10: 2K, Resistor_THT:R_Axial_DIN0204_L3.6mm_D1.6mm_P5.08mm_Horizontal, symbol Device:R_US
- added R11: 470, Resistor_THT:R_Axial_DIN0204_L3.6mm_D1.6mm_P5.08mm_Horizontal, symbol Device:R_US
- added R12: 220, Resistor_THT:R_Axial_DIN0204_L3.6mm_D1.6mm_P5.08mm_Horizontal, symbol Device:R_US
- CURRENT_SENSOR1, DHT1, VOLTAGE_SENSOR1: footprint Connector:FanPinHeader_1x03_P2.54mm_Vertical -> Connector_PinHeader_2.54mm:PinHeader_1x03_P2.54mm_Vertical
- DC_MOTOR_DELIVERY1, LDR1, LDR2, LDR3, LDR4, WATER_LEVEL_SW1, WATER_PUMP1: footprint TerminalBlock:TerminalBlock_bornier-2_P5.08mm -> KF301-2P:KF301-2P
- DS18B1, SERVO1, SERVO2: footprint TerminalBlock:TerminalBlock_bornier-3_P5.08mm -> KF301-3P:KF301-3P
- FC-28-MOD1, MQ9-GAS-SENSOR1: footprint Connector:FanPinHeader_1x04_P2.54mm_Vertical -> Connector_PinHeader_2.54mm:PinHeader_1x04_P2.54mm_Vertical
- U1: footprint esp32_devkit_v1_doit:esp32_devkit_v1_doit -> ESP3_DEVKIT_30PIN:esp32_devkit_v1_doit
Connections:
- net +12V: now also 12V_PWR1.1 (Pin_1), MP2482MOD1.2 (VCC), NPK_SEN1.4 (Pin_4), R10.1
- net +3V3: now also R12.1
- net +5V: now also MAX485MOD1.4 (VCC), MP2482MOD1.3 (5V), R11.1
- net DI_SIGNAL: now also MAX485MOD1.8 (DI)
- net GND: now also 12V_PWR1.2 (Pin_2), D3.1 (K), D4.1 (K), D5.1 (K), MAX485MOD1.1 (GND), MP2482MOD1.1 (GND), MP2482MOD1.4 (GND), NPK_SEN1.3 (Pin_3)
- net RE_SIGNAL: now also MAX485MOD1.6 (RE), MAX485MOD1.7 (DE)
- net RO_SIGNAL: now also MAX485MOD1.5 (RO)
- new net: D4.2 (A), R11.2
- new net: D3.2 (A), R10.2
- new net: D5.2 (A), R12.2
- new net A: MAX485MOD1.2 (A), NPK_SEN1.2 (Pin_2)
- new net B: MAX485MOD1.3 (B), NPK_SEN1.1 (Pin_1)
Other:
- moved on the sheet: CURRENT_SENSOR1, D1, D2, DC_MOTOR_DELIVERY1, DHT1, DS18B1, FC-28-MOD1, LDR1, LDR2, LDR3, LDR4, MQ9-GAS-SENSOR1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
